Commit message: Initial upload

File: elfin3/elfin3_ros2_gazebo/urdf/elfin3_gazebo.xacro (robot description, xacro)
@@ -1,7 +1,12 @@
 <?xml version="1.0"?>
+<!--
+  ROS2 Humble migration:
+    - fake_components/GenericSystem -> mock_components/GenericSystem
+      (fake_components was renamed in Humble; the old name is gone)
+-->
 <robot xmlns:xacro="http://www.ros.org/wiki/xacro">
   <xacro:macro name="elfin3_gazebo"
     params="use_fake_hardware:=false
-    use_real_hardware:=true">
+            use_real_hardware:=true">
     <gazebo>
       <plugin filename="libgazebo_ros2_control.so" name="gazebo_ros2_control">
@@ -17,5 +22,6 @@
         <xacro:unless value="${use_real_hardware}">
           <xacro:if value="${use_fake_hardware}">
-              <plugin>fake_components/GenericSystem</plugin>
+            <!-- Humble: fake_components -> mock_components -->
+            <plugin>mock_components/GenericSystem</plugin>
           </xacro:if>
           <xacro:unless value="${use_fake_hardware}">
@@ -97,24 +103,24 @@
       </joint>
     </ros2_control>
- <gazebo reference="elfin_link2">
-    <visual name='visual'>
-     <material>
-       <script>
-         <uri>file://media/materials/scripts/gazebo.material</uri>
-         <name>Gazebo/Grey</name>
-       </script>
-     </material>
-    </visual>
-  </gazebo>
-  <gazebo reference="elfin_link4">
-    <visual name='visual'>
-     <material>
-       <script>
-         <uri>file://media/materials/scripts/gazebo.material</uri>
-         <name>Gazebo/Grey</name>
-       </script>
-     </material>
-    </visual>
-  </gazebo>
+    <gazebo reference="elfin_link2">
+      <visual name='visual'>
+        <material>
+          <script>
+            <uri>file://media/materials/scripts/gazebo.material</uri>
+            <name>Gazebo/Grey</name>
+          </script>
+        </material>
+      </visual>
+    </gazebo>
+    <gazebo reference="elfin_link4">
+      <visual name='visual'>
+        <material>
+          <script>
+            <uri>file://media/materials/scripts/gazebo.material</uri>
+            <name>Gazebo/Grey</name>
+          </script>
+        </material>
+      </visual>
+    </gazebo>
   </xacro:macro>
 </robot>

File: elfin3/elfin3_ros2_gazebo/urdf/elfin3_transmission.xacro (robot description, xacro)
@@ -1,10 +1,16 @@
 <?xml version="1.0"?>
+<!--
+  ROS2 Humble migration:
+    Removed <hardwareInterface>hardware_interface/PositionJointInterface</hardwareInterface>
+    tags. These were used by gazebo_ros_control in ROS1; gazebo_ros2_control
+    instead reads everything from the <ros2_control> block in elfin3_gazebo.xacro.
+    The <transmission> blocks themselves are kept (and stripped down) because
+    some downstream tools still parse them; they are otherwise a no-op.
+-->
 <robot xmlns:xacro="http://wiki.ros.org/xacro">
-  <xacro:macro name="elfin3_transmission" >
-     <transmission name="elfin_joint1_trans">
+  <xacro:macro name="elfin3_transmission">
+    <transmission name="elfin_joint1_trans">
       <type>transmission_interface/SimpleTransmission</type>
-      <joint name="elfin_joint1">
-        <hardwareInterface>hardware_interface/PositionJointInterface</hardwareInterface>
-      </joint>
+      <joint name="elfin_joint1"/>
       <actuator name="elfin_joint1_motor">
         <mechanicalReduction>1</mechanicalReduction>
@@ -13,7 +19,5 @@
     <transmission name="elfin_joint2_trans">
       <type>transmission_interface/SimpleTransmission</type>
-      <joint name="elfin_joint2">
-        <hardwareInterface>hardware_interface/PositionJointInterface</hardwareInterface>
-      </joint>
+      <joint name="elfin_joint2"/>
       <actuator name="elfin_joint2_motor">
         <mechanicalReduction>1</mechanicalReduction>
@@ -22,7 +26,5 @@
     <transmission name="elfin_joint3_trans">
       <type>transmission_interface/SimpleTransmission</type>
-      <joint name="elfin_joint3">
-        <hardwareInterface>hardware_interface/PositionJointInterface</hardwareInterface>
-      </joint>
+      <joint name="elfin_joint3"/>
       <actuator name="elfin_joint3_motor">
         <mechanicalReduction>1</mechanicalReduction>
@@ -31,7 +33,5 @@
     <transmission name="elfin_joint4_trans">
       <type>transmission_interface/SimpleTransmission</type>
-      <joint name="elfin_joint4">
-        <hardwareInterface>hardware_interface/PositionJointInterface</hardwareInterface>
-      </joint>
+      <joint name="elfin_joint4"/>
       <actuator name="elfin_joint4_motor">
         <mechanicalReduction>1</mechanicalReduction>
@@ -40,7 +40,5 @@
     <transmission name="elfin_joint5_trans">
       <type>transmission_interface/SimpleTransmission</type>
-      <joint name="elfin_joint5">
-        <hardwareInterface>hardware_interface/PositionJointInterface</hardwareInterface>
-      </joint>
+      <joint name="elfin_joint5"/>
       <actuator name="elfin_joint5_motor">
         <mechanicalReduction>1</mechanicalReduction>
@@ -49,7 +47,5 @@
     <transmission name="elfin_joint6_trans">
       <type>transmission_interface/SimpleTransmission</type>
-      <joint name="elfin_joint6">
-        <hardwareInterface>hardware_interface/PositionJointInterface</hardwareInterface>
-      </joint>
+      <joint name="elfin_joint6"/>
       <actuator name="elfin_joint6_motor">
         <mechanicalReduction>1</mechanicalReduction>
